File: hardware/rupter.kicad_pcb (KiCad board)
At the start: 2 copper layers, 100 x 40 mm, 32 parts, among them J1 rca, J2 rca, J3 Barrel_Jack_Switch, SW1 SPDT, SW2 SPDT, SW3 SPDT, SW4 SPDT, SW5 SPDT, SW6 SPDT, SW7 SPDT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

Commit message: latest circuit revision
Parts:
- J3: footprint Connector_BarrelJack:BarrelJack_Horizontal -> lib_fp:BarrelJack_Horizontal
