File: hardware/_rupture_.kicad_pcb (KiCad board)
At the start: 2 copper layers, 100 x 40 mm, 32 parts, among them J1 rca, J2 rca, J3 Barrel_Jack_Switch, SW1 SPDT, SW2 SPDT, SW3 SPDT, SW4 SPDT, SW5 SPDT, SW6 SPDT, SW7 SPDT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

Commit message: update bom
Other:
- board text added: "JLCJLCJLCJLC"

Commit message: update with panels
Other:
- net class Default removed
